Commit message: My custom config, launch, and URDF files for recon_bot

File: zed_wrapper/urdf/zed_macro.urdf.xacro (robot description, xacro)
@@ -129,4 +129,12 @@
       <origin xyz="${optical_offset_x} ${baseline/2} 0" rpy="0 0 0" />
     </joint>
+    <!-- เพิ่มตรงนี้! -->
+    <link name="${name}_imu_link" />
+    <joint name="${name}_imu_joint" type="fixed">
+      <parent link="${name}_left_camera_frame"/>
+      <child link="${name}_imu_link"/>
+      <origin xyz="0.0 0.0 0.0" rpy="0 0 0" />
+    </joint>
+    <!-- จบการเพิ่ม -->
     <link name="${name}_left_camera_optical_frame"/>
     <joint name="${name}_left_camera_optical_joint" type="fixed">
